File: board/industrial_input.sch (KiCad schematic (older format))
At the start: 3 parts

Commit message: Industrial Input Schematic Notes
Other:
- note added: "0.7mA @ 24V Input, 210mV drop on Schottky array"
- note added: "48kHz Single Pole Low Pass Filter"
Changed lines of the file:
@@
 Wire Wire Line
 	6100 4250 6200 4250
+Text Notes 5000 3600 0    60   ~ 0
+48kHz Single Pole Low Pass Filter
+Text Notes 5000 3700 0    60   ~ 0
+0.7mA @ 24V Input, 210mV drop on Schottky array
 $EndSCHEMATC
