File: board/robot_controller.kicad_pcb (KiCad board)
At the start: 2 copper layers, 294 parts, among them J104 JTAG-ARM, J111 UEXT, J112 UEXT, J201 CONN_2, J2301 CONN_STEPPER, J2401 CONN_STEPPER, J2501 CONN_STEPPER, J2601 CONN_STEPPER, J301 CONN_2, P102 CONN_1, P103 CONN_1, P104 CONN_1, P105 CONN_1, P106 CONN_1, P107 CONN_1, P108 CONN_1, P109 CONN_1, P110 CONN_1, P111 CONN_1, P112 CONN_1, P113 CONN_1, P114 CONN_1, P115 CONN_1, P116 CONN_1, P117 CONN_1, P118 CONN_1, P119 CONN_1, P120 CONN_1, P121 CONN_1, P122 CONN_1, P123 CONN_1, P124 CONN_1, P125 CONN_1, P126 CONN_1, P127 CONN_1, P128 CONN_1, P129 CONN_1, P130 CONN_1, Q101 PNP, Q1501 NJT4031NT1G, Q1601 NJT4031NT1G, Q1701 NJT4031NT1G, Q1801 NJT4031NT1G, Q1901 NJT4031NT1G, Q2001 NJT4031NT1G, Q2101 NJT4031NT1G, Q2201 NJT4031NT1G, Q401 MMBT5962, Q402 MMBT5962, Q501 MMBT5962, Q502 MMBT5962, U101 STM32F405-144, U102 FT232RL, U201 MAX6675, U2301 L6470, U2401 L6470, U2501 L6470, U2601 L6470, U301 MAX6675, U601 LMZ14201, X101 8MHZ

Commit message: Started layout of a few other 'modules'. More work on the stepper drivers. Used more Andrew footprints.
Parts:
- added J106: USBCONN, Connect:USB_B, F.Cu at (155.7, -67.5)
- added J109: USBCONN, Connect:USB_B, F.Cu at (0.00, 0.00)
- added J2302: CONN_2, components:CONN_TEMP, F.Cu at (6.35, 17.5)
- added J2402: CONN_2, components:CONN_TEMP, F.Cu at (21.6, 12.4)
- added J2502: CONN_2, components:CONN_TEMP, F.Cu at (24.8, 3.17)
- added J2602: CONN_2, components:CONN_TEMP, F.Cu at (37.5, 6.67)
- moved D106 257.2 mm to (160.5, -80.5), turned to 90 degrees
- moved D107 254.1 mm to (158.6, -80.5), turned to 90 degrees
- moved R123 254.0 mm to (158.6, -77.6), turned to 270 degrees
- moved R121 249.5 mm to (160.5, -77.6), turned to 270 degrees
- moved U102 192.5 mm to (155.7, -86.8), turned to 180 degrees
- moved C130 192.0 mm to (155.7, -80.5), turned to 270 degrees
- moved D109 183.4 mm to (196.2, -68.3), turned to 90 degrees
- moved U601 173.2 mm to (170.8, -81.0)
- moved R112 172.7 mm to (252.4, 96.8)
- moved R128 169.5 mm to (195.3, -65.7)
- moved Q1501 167.3 mm to (192.7, 52.1)
- moved R124 162.6 mm to (149.1, -89.4), turned to 270 degrees
- moved R126 160.1 mm to (188.9, -59.4), turned to 180 degrees
- moved C132 158.7 mm to (158.0, -93.2), turned to 90 degrees
- moved C129 152.9 mm to (194.6, -63.2), turned to 90 degrees
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Routing:
- net +3.3V: track 72.2 -> 115.4 mm
- net GND: track 152.2 -> 184.6 mm, vias 53 -> 61
- net (no net): track 42.7 -> 72.7 mm
- net /Stepper 0/STCK: track 5.13 -> 22.7 mm, vias 1 -> 2
- net Net-(J106-Pad3): track 0.00 -> 14.6 mm
- net +5V: track 0.00 -> 13.2 mm
- net /Stepper 0/ADCIN: track 65.7 -> 78.7 mm
- net /Stepper 0/~CS: track 9.31 -> 22.2 mm, vias 1 -> 2
- net Net-(J106-Pad2): track 0.00 -> 12.5 mm
- net /Stepper 0/SDO: track 8.14 -> 20.6 mm, vias 1 -> 2
- net /Stepper 0/SDI: track 8.99 -> 20.6 mm, vias 1 -> 2
- net /Stepper 0/SCK: track 9.75 -> 20.7 mm, vias 1 -> 2
- net Net-(C601-Pad2): track 0.00 -> 7.12 mm
- net /Stepper 0/OSCIN: track 63.2 -> 68.5 mm
- net /Stepper 1/OSCIN: track 64.2 -> 69.4 mm
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
Commit message: More components layed out
Parts:
- added J107: CONN_8, components:SCONN_8, F.Cu at (99.1, -87.6)
- added J108: CONN_8, components:SCONN_8, F.Cu at (43.8, -87.6)
- moved J109 219.7 mm to (174.3, 133.7)
- moved Q1501 218.2 mm to (17.1, -77.5)
- moved D1501 217.9 mm to (17.1, -67.6), turned to 270 degrees
- moved R1201 217.3 mm to (106.7, -77.8), turned to 270 degrees
- moved D1601 217.2 mm to (24.8, -67.6), turned to 270 degrees
- moved R701 215.5 mm to (81.3, -77.8), turned to 270 degrees
- moved C1201 215.3 mm to (106.7, -72.7)
- moved R1401 214.2 mm to (116.8, -77.8), turned to 270 degrees
- moved C701 213.3 mm to (81.3, -72.7)
- moved R1601 212.8 mm to (22.5, -62.9), turned to 90 degrees
- moved C1401 212.6 mm to (116.8, -72.7)
- moved R1501 212.4 mm to (14.9, -62.9), turned to 90 degrees
- moved R1301 212.3 mm to (111.8, -77.8), turned to 270 degrees
- moved R1101 212.0 mm to (101.6, -77.8), turned to 270 degrees
- moved D1801 211.8 mm to (40.0, -67.6), turned to 270 degrees
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Routing:
- net +3.3V: track 115.4 -> 162.5 mm, vias 2 -> 10
- net +24V: track 262.0 -> 285.2 mm, vias 40 -> 48
- net /Industrial Output 0/Sink: track 0.00 -> 22.4 mm
- net /Industrial Output 7/Sink: track 0.00 -> 22.4 mm
- net /Industrial Output 6/Sink: track 0.00 -> 20.1 mm
- net /Industrial Output 1/Sink: track 0.00 -> 20.1 mm
- net /Industrial Output 2/Sink: track 0.00 -> 19.1 mm
- net /Industrial Output 5/Sink: track 0.00 -> 19.1 mm
- net /Industrial Output 4/Sink: track 0.00 -> 18.0 mm
- net /Industrial Output 3/Sink: track 0.00 -> 18.0 mm
- net GND: track 184.6 -> 196.3 mm, vias 61 -> 69
- net Net-(Q2201-Pad2): track 0.00 -> 10.6 mm
- net Net-(Q1901-Pad2): track 0.00 -> 10.6 mm
- net Net-(Q1701-Pad2): track 0.00 -> 10.6 mm
- net Net-(Q1601-Pad2): track 0.00 -> 10.6 mm
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
Commit message: Made use of new components
Parts:
- added J101: CONN_2, components:SCONN_2, F.Cu at (127.0, -87.6)
- added J102: CONN_2, components:SCONN_2, F.Cu at (15.2, -87.6)
- added J103: CONN_2, components:SCONN_2, F.Cu at (71.1, -87.6)
- added J105: CONN_2, components:PWRSCONN_2, F.Cu at (-33.3, -24.1)
- added J110: CONN_4, Pin_Headers:Pin_Header_Straight_1x04, F.Cu at (87.9, 77.5)
- added P101: CONN_4, components:SCONN_4, F.Cu at (229.6, 46.4)
- J106, J109: footprint Connect:USB_B -> components:USB_B
- J201, J2302, J2402, J2502, J2602, J301: footprint components:CONN_TEMP -> components:SCONN_2
- R127: footprint Potentiometers:Potentiometer_VishaySpectrol-Econtrim-Type36M -> components:TRIMMER_POT
- moved J2302 296.8 mm to (273.4, 147.0)
- moved R127 219.3 mm to (-21.3, -3.81)
- moved D108 216.2 mm to (-9.21, 4.13)
- moved D109 216.2 mm to (-9.21, -0.95)
- moved R125 216.2 mm to (-8.89, 7.62)
- moved C129 216.2 mm to (-10.8, 4.13)
- moved C136 216.2 mm to (-10.8, -0.95)
- moved R122 216.2 mm to (-10.8, 7.62)
- moved R126 216.2 mm to (-16.5, 7.94)
- moved R128 216.2 mm to (-10.2, 1.59)
- moved J2502 185.5 mm to (142.2, 146.7)
- moved C601 182.4 mm to (-7.62, -57.5)
- moved C602 182.4 mm to (-3.81, -62.2)
- moved C603 182.4 mm to (-11.1, -49.2)
- moved C604 182.4 mm to (-11.1, -57.5)
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Connections:
- Q1501 pad 1: GNDPWR -> GND
- Q1601 pad 1: GNDPWR -> GND
- Q1701 pad 1: GNDPWR -> GND
- Q1801 pad 1: GNDPWR -> GND
- Q1901 pad 1: GNDPWR -> GND
- Q2001 pad 1: GNDPWR -> GND
- Q2101 pad 1: GNDPWR -> GND
- Q2201 pad 1: GNDPWR -> GND
Routing:
- net +24V: track 285.2 -> 373.3 mm, vias 48 -> 49
- net +3.3V: track 162.5 -> 199.3 mm
- net Net-(J106-Pad3): track 14.6 -> 0.00 mm
- net GND: track 196.3 -> 210.8 mm, vias 69 -> 77
- net Net-(J106-Pad2): track 12.5 -> 0.00 mm
- net +5V: track 13.2 -> 5.34 mm
- net /Stepper 0/ADCIN: track 78.7 -> 72.9 mm
- net /Temp Sensor 0/~CS: track 0.00 -> 4.95 mm
- net /Temp Sensor 1/~CS: track 0.00 -> 4.87 mm
- net Net-(R126-Pad2): track 4.53 -> 0.00 mm
- net Net-(R127-Pad3): track 3.86 -> 0.00 mm
- net Net-(C133-Pad1): track 2.11 -> 0.25 mm
- net Net-(D107-Pad2): track 4.13 -> 5.61 mm
- net Net-(D106-Pad2): track 5.18 -> 3.71 mm
Other:
- rule pad_to_mask_clearance: 0.2032 -> 0.2
