File: board/industrial_output.sch (KiCad schematic (older format))
At the start: 3 parts, among them Q1501 NJT4031NT1G

Commit message: Layed out in general where stuff is going to be located.
Changed lines of the file:
@@
 AR Path="/52FAF275/52E6FDE0" Ref="Q2101"  Part="1"
 AR Path="/52FAF279/52E6FDE0" Ref="Q2201"  Part="1"
-F 0 "Q1501" H 5650 4500 50  0000 L CNN
+F 0 "Q2201" H 5650 4500 50  0000 L CNN
 F 1 "NJT4031NT1G" H 5650 4600 50  0000 L CNN
 F 2 "" H 5450 4500 60  0000 C CNN
@@
 AR Path="/52FAF275/52E6FDF4" Ref="R2101"  Part="1"
 AR Path="/52FAF279/52E6FDF4" Ref="R2201"  Part="1"
-F 0 "R1501" V 4980 4500 50  0000 C CNN
+F 0 "R2201" V 4980 4500 50  0000 C CNN
 F 1 "470" V 4900 4500 50  0000 C CNN
 F 2 "" H 4900 4500 60  0000 C CNN
@@
 AR Path="/52FAF275/52E705F0" Ref="D2101"  Part="1"
 AR Path="/52FAF279/52E705F0" Ref="D2201"  Part="1"
-F 0 "D1501" V 5900 3800 40  0000 R CNN
+F 0 "D2201" V 5900 3800 40  0000 R CNN
 F 1 "RSX501L-20TE25" V 5800 3800 40  0001 R CNN
 F 2 "" H 5800 3900 60  0000 C CNN
@@
 Connection ~ 5550 4200
 $Comp
-L +24V #PWR0164
+L +24V #PWR1501
 U 1 1 52E70673
 P 5800 3600
-AR Path="/52FAAFCB/52E70673" Ref="#PWR0164"  Part="1"
-AR Path="/52FAC46B/52E70673" Ref="#PWR0166"  Part="1"
-AR Path="/52FAD3BD/52E70673" Ref="#PWR0168"  Part="1"
-AR Path="/52FAD3C1/52E70673" Ref="#PWR0170"  Part="1"
-AR Path="/52FAF26D/52E70673" Ref="#PWR0172"  Part="1"
-AR Path="/52FAF271/52E70673" Ref="#PWR0174"  Part="1"
-AR Path="/52FAF275/52E70673" Ref="#PWR0176"  Part="1"
-AR Path="/52FAF279/52E70673" Ref="#PWR0178"  Part="1"
-F 0 "#PWR0178" H 5800 3550 20  0001 C CNN
+AR Path="/52FAAFCB/52E70673" Ref="#PWR1501"  Part="1"
+AR Path="/52FAC46B/52E70673" Ref="#PWR1601"  Part="1"
+AR Path="/52FAD3BD/52E70673" Ref="#PWR1701"  Part="1"
+AR Path="/52FAD3C1/52E70673" Ref="#PWR1801"  Part="1"
+AR Path="/52FAF26D/52E70673" Ref="#PWR1901"  Part="1"
+AR Path="/52FAF271/52E70673" Ref="#PWR2001"  Part="1"
+AR Path="/52FAF275/52E70673" Ref="#PWR2101"  Part="1"
+AR Path="/52FAF279/52E70673" Ref="#PWR2201"  Part="1"
+F 0 "#PWR2201" H 5800 3550 20  0001 C CNN
 F 1 "+24V" H 5800 3700 30  0000 C CNN
 F 2 "" H 5800 3600 60  0000 C CNN
@@
 	5550 4700 5550 4800
 $Comp
-L GND #PWR0165
+L GND #PWR1502
 U 1 1 5312BB8B
 P 5550 4800
-AR Path="/52FAAFCB/5312BB8B" Ref="#PWR0165"  Part="1"
-AR Path="/52FAC46B/5312BB8B" Ref="#PWR0167"  Part="1"
-AR Path="/52FAD3BD/5312BB8B" Ref="#PWR0169"  Part="1"
-AR Path="/52FAD3C1/5312BB8B" Ref="#PWR0171"  Part="1"
-AR Path="/52FAF26D/5312BB8B" Ref="#PWR0173"  Part="1"
-AR Path="/52FAF271/5312BB8B" Ref="#PWR0175"  Part="1"
-AR Path="/52FAF275/5312BB8B" Ref="#PWR0177"  Part="1"
-AR Path="/52FAF279/5312BB8B" Ref="#PWR0179"  Part="1"
-F 0 "#PWR0179" H 5550 4800 30  0001 C CNN
+AR Path="/52FAAFCB/5312BB8B" Ref="#PWR1502"  Part="1"
+AR Path="/52FAC46B/5312BB8B" Ref="#PWR1602"  Part="1"
+AR Path="/52FAD3BD/5312BB8B" Ref="#PWR1702"  Part="1"
+AR Path="/52FAD3C1/5312BB8B" Ref="#PWR1802"  Part="1"
+AR Path="/52FAF26D/5312BB8B" Ref="#PWR1902"  Part="1"
+AR Path="/52FAF271/5312BB8B" Ref="#PWR2002"  Part="1"
+AR Path="/52FAF275/5312BB8B" Ref="#PWR2102"  Part="1"
+AR Path="/52FAF279/5312BB8B" Ref="#PWR2202"  Part="1"
+F 0 "#PWR2202" H 5550 4800 30  0001 C CNN
 F 1 "GND" H 5550 4730 30  0001 C CNN
 F 2 "" H 5550 4800 60  0000 C CNN
